File: hardware/EnphaseLimiter_HardwareDesign/EnphaseLimiter_HardwareDesign.kicad_sch (KiCad schematic)
At the start: 30 parts, among them J1 Conn_01x02, J2 Conn_01x06, J3 Conn_01x05, J4 Conn_01x05, K1 Relay_SPST-NO, K2 Relay_SPST-NO, K3 Relay_SPST-NO, K4 Relay_SPST-NO, Q1 2N7000, Q2 2N7000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

Commit message: Corrected schematic design errors on relay drive
Connections:
- net +12V: now also D1.1 (K), D2.1 (K), D3.1 (K), D4.1 (K), K1.A1, K2.A1, K3.A1, K4.A1
- net Drive1: now also D1.2 (A), K1.A2; no longer D1.1 (K), K1.A1
- net Drive2: now also D2.2 (A), K2.A2; no longer D2.1 (K), K2.A1
- net Drive3: now also D3.2 (A), K3.A2; no longer D3.1 (K), K3.A1
- net Drive4: now also D4.2 (A), K4.A2; no longer D4.1 (K), K4.A1
- net GND: no longer D1.2 (A), D2.2 (A), D3.2 (A), D4.2 (A), K1.A2, K2.A2, K3.A2, K4.A2
